File: Hardware/Qwiic_Relay.brd (EAGLE design)
At the start: 25.4 x 50.8 mm, 34 parts, among them J2 Qwiic Right Angle, J3 Qwiic Right Angle, J4 AVR_SPI_PROG_3X2TESTPOINTS, Q4 600mA/40V, U1 ATTIN85_SOIC_5.3MM, U2 OPTO_ISOLATOR_DIP

Commit message: ordered board
Connections:
- net MISO: now also U1.6; no longer U1.7
- net SCL: now also U1.7; no longer U1.2
- net SDA: now also U1.5; no longer U1.6
Routing:
- net SDA: track 36.5 -> 46.0 mm, vias 1 -> 3
- net MISO: track 0.00 -> 4.89 mm, vias 0 -> 1
- net 3.3V: track 70.8 -> 75.2 mm
- net GND: track 20.6 -> 24.1 mm, vias 2 -> 4
- net SCL: track 25.5 -> 26.2 mm, vias 2 -> 0
Other:
- board text added: "x11"
- board text removed: "v2"
