File: Hardware/Qwiic_Relay.sch (EAGLE design)
At the start: 34 parts, among them J2 Qwiic Right Angle, J3 Qwiic Right Angle, J4 AVR_SPI_PROG_3X2TESTPOINTS, Q4 600mA/40V, U1 ATTIN85_SOIC_5.3MM, U2 OPTO_ISOLATOR_DIP

Commit message: updated repo
- Removed unnecessary eagle documents
- added IoT relay as related product
- included a pdf of the schematic
- added relay datasheet
Other:
- note removed: "2222 or can we go lower?"
- note removed: "remove this 10 ohm and check that you don't need it"
Changed lines of the file:
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@@
 <setting verticaltext="up"/>
 </settings>
-<grid distance="0.05" unitdist="inch" unit="inch" style="lines" multiple="1" display="yes" altdistance="0.005" altunitdist="inch" altunit="inch"/>
+<grid distance="0.1" unitdist="inch" unit="inch" style="lines" multiple="1" display="no" altdistance="0.01" altunitdist="inch" altunit="inch"/>
 <layers>
 <layer number="1" name="Top" color="4" fill="1" visible="no" active="no"/>
@@
 <text x="169.164" y="109.728" size="2.032" layer="97" align="top-left">I2C Port</text>
 <wire x1="147.32" y1="99.06" x2="248.92" y2="99.06" width="0.2032" layer="97" style="longdash"/>
-<text x="38.1" y="175.26" size="2.54" layer="91">remove this 10 ohm
-and check that you don't need it</text>
-<text x="99.06" y="114.3" size="1.27" layer="91">2222 or can we go lower?</text>
 </plain>
 <instances>
@@
 </schematic>
 </drawing>
-<compatibility>
-<note version="6.3" minversion="6.2.2" severity="warning">
-Since Version 6.2.2 text objects can contain more than one line,
-which will not be processed correctly with this version.
-</note>
-</compatibility>
 </eagle>

Commit message: added pdf
added pdf of schematic into the hardware folder,changed read me, and added more details to the schematic about max currents.
Other:
- note added: "The board is designed for a 15*C temperature rise Allowing for a continous current draw of 5.5A. The relay can handle 10 A at 110VAC for short pulses (under 20 seconds)."
Changed lines of the file:
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@@
 <text x="169.164" y="109.728" size="2.032" layer="97" align="top-left">I2C Port</text>
 <wire x1="147.32" y1="99.06" x2="248.92" y2="99.06" width="0.2032" layer="97" style="longdash"/>
+<text x="15.24" y="170.18" size="1.27" layer="97">The board is designed for a 15*C temperature
+rise Allowing for a continous current draw of
+5.5A. The relay can handle 10 A at 110VAC
+for short pulses (under 20 seconds).</text>
 </plain>
 <instances>
@@
 </schematic>
 </drawing>
+<compatibility>
+<note version="6.3" minversion="6.2.2" severity="warning">
+Since Version 6.2.2 text objects can contain more than one line,
+which will not be processed correctly with this version.
+</note>
+</compatibility>
 </eagle>

Commit message: Rev 2 and sent to fab
Revision 2 of the board. (x12)

added more clearance to the PCB
added buzzard labels
added cutout into the dimension layer so that it is exported to GKO

fixed spacing on the Schematic
added address jumper to pin 2 of the ATtiny85

on the panel sent off to production
- labeled the cutout as "cutout" in the GKO
Parts:
- added JP10: JUMPER-SMT_2_NO_NO-SILK, SparkFun-Jumpers:JUMPER-SMT_2_NO_NO-SILK
- K1: device Relay_SPDT:RELAY_SPDT_1C -> SparkX:RELAY_SPDT_1C
- U2: value OPTO_ISOLATOR_DIP -> OPTO_ISOLATOR; device LTV-816:OPTO_ISOLATOR_DIP -> SparkX:OPTO_ISOLATOR_SMD
Connections:
- new net N$5: JP10.1, U1.(PCINT3/XTAL1/CLKI/OC1B/ADC3)PB3
- net GND: now also JP10.2
- net NC: now also J5.1; no longer J5.3
- net NO: now also J5.3; no longer J5.1
Other:
- note added: "ADDR Open - Default Address 0x18 Closed - 0x19 Address is configurable in software"
- moved on the sheet: J5, R2

Commit message: Matching components values
Parts:
- R1: device SparkFun-Resistors:47KOHM-0603-1/10W-1% -> SparkFun-Resistors:10OHM-0603-1/10W-5%
- R2: value 100 -> 330; device SparkFun-Resistors:100OHM-0603-1/4W-5% -> SparkFun-Resistors:330OHM-0603-1/10W-1%
- R4: device SparkFun-Resistors:300OHM-0603-1/10W-1% -> SparkFun-Resistors:330OHM-0603-1/10W-1%
- R6, R7: value 2.2K -> 2.2k; device SparkFun-Resistors:4.7KOHM-0603-1/10W-1% -> SparkFun-Resistors:2.2KOHM-0603-1/10W-1%
- R8: value 10K -> 10k; device SparkFun-Resistors:330OHM-0603-1/10W-1% -> SparkFun-Resistors:10KOHM-0603-1/10W-1%
- R9: device SparkFun-Resistors:330OHM-0603-1/10W-1% -> SparkFun-Resistors:1KOHM-0603-1/10W-1%
Changed lines of the file:
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@@
 <?xml version="1.0" encoding="utf-8"?>
 <!DOCTYPE eagle SYSTEM "eagle.dtd">
-<eagle version="7.7.0">
+<eagle version="9.0.0">
 <drawing>
 <settings>
-<setting alwaysvectorfont="yes"/>
+<setting alwaysvectorfont="no"/>
+<setting keepoldvectorfont="yes"/>
 <setting verticaltext="up"/>
 </settings>
@@
 <part name="FRAME1" library="SparkFun-Aesthetics" deviceset="FRAME-LETTER" device=""/>
 <part name="GND1" library="SparkFun-PowerSymbols" deviceset="GND" device=""/>
-<part name="R2" library="SparkFun-Resistors" deviceset="100OHM" device="-0603-1/4W-5%" value="100"/>
+<part name="R2" library="SparkFun-Resistors" deviceset="330OHM" device="-0603-1/10W-1%" value="330"/>
 <part name="GND2" library="SparkFun-PowerSymbols" deviceset="GND" device=""/>
 <part name="GND3" library="SparkFun-PowerSymbols" deviceset="GND" device=""/>
@@
 <part name="SUPPLY6" library="SparkFun-PowerSymbols" deviceset="VCC" device="" value="3.3V"/>
 <part name="D2" library="SparkFun-LED" deviceset="LED-BLUE" device="0603" value="BLUE"/>
-<part name="R4" library="SparkFun-Resistors" deviceset="300OHM" device="-0603-1/10W-1%" value="330"/>
+<part name="R4" library="SparkFun-Resistors" deviceset="330OHM" device="-0603-1/10W-1%" value="330"/>
 <part name="GND5" library="SparkFun-PowerSymbols" deviceset="GND" device=""/>
 <part name="C1" library="SparkFun-Capacitors" deviceset="10UF" device="-0603-6.3V-20%" value="10uF"/>
@@
 <part name="GND6" library="SparkFun-PowerSymbols" deviceset="GND" device=""/>
 <part name="SUPPLY7" library="SparkFun-PowerSymbols" deviceset="VCC" device="" value="3.3V"/>
-<part name="R1" library="SparkFun-Resistors" deviceset="47KOHM" device="-0603-1/10W-1%" value="10"/>
+<part name="R1" library="SparkFun-Resistors" deviceset="10OHM" device="-0603-1/10W-5%" value="10"/>
 <part name="U$3" library="SparkX" deviceset="SPARKX-LOGO" device="4"/>
 <part name="LOGO1" library="SparkFun-Aesthetics" deviceset="OSHW-LOGO" device="MINI"/>
@@
 <part name="JP2" library="SparkFun" deviceset="FIDUCIAL" device="UFIDUCIAL"/>
 <part name="JP6" library="SparkFun" deviceset="FIDUCIAL" device="UFIDUCIAL"/>
-<part name="R6" library="SparkFun-Resistors" deviceset="4.7KOHM" device="-0603-1/10W-1%" value="2.2K"/>
-<part name="R7" library="SparkFun-Resistors" deviceset="4.7KOHM" device="-0603-1/10W-1%" value="2.2K"/>
+<part name="R6" library="SparkFun-Resistors" deviceset="2.2KOHM" device="-0603-1/10W-1%" value="2.2k"/>
+<part name="R7" library="SparkFun-Resistors" deviceset="2.2KOHM" device="-0603-1/10W-1%" value="2.2k"/>
 <part name="JP7" library="SparkFun-Jumpers" deviceset="JUMPER-SMT_3_2-NC_PASTE" device="_SILK" value=""/>
 <part name="SUPPLY9" library="SparkFun-PowerSymbols" deviceset="3.3V" device=""/>
 <part name="J4" library="SparkFun-Connectors" deviceset="AVR_SPI_PROG_3X2" device="TESTPOINTS"/>
-<part name="R8" library="SparkFun-Resistors" deviceset="330OHM" device="-0603-1/10W-1%" value="10K"/>
+<part name="R8" library="SparkFun-Resistors" deviceset="10KOHM" device="-0603-1/10W-1%" value="10k"/>
 <part name="SUPPLY10" library="SparkFun-PowerSymbols" deviceset="3.3V" device=""/>
-<part name="R9" library="SparkFun-Resistors" deviceset="330OHM" device="-0603-1/10W-1%" value="1k"/>
+<part name="R9" library="SparkFun-Resistors" deviceset="1KOHM" device="-0603-1/10W-1%" value="1k"/>
 <part name="D3" library="SparkFun-LED" deviceset="LED-RED" device="0603" value="RED"/>
 <part name="SUPPLY11" library="SparkFun-PowerSymbols" deviceset="3.3V" device=""/>
