File: Hardware/Production/Qwiic_Relay-Panel.brd (EAGLE design)
At the start: 103.1 x 138.2 mm, 297 parts, among them J11 Qwiic Right Angle, J12 Qwiic Right Angle, J13 AVR_SPI_PROG_3X2TESTPOINTS, J16 Qwiic Right Angle, J17 Qwiic Right Angle, J18 AVR_SPI_PROG_3X2TESTPOINTS, J2 Qwiic Right Angle, J21 Qwiic Right Angle, J22 Qwiic Right Angle, J23 AVR_SPI_PROG_3X2TESTPOINTS, J26 Qwiic Right Angle, J27 Qwiic Right Angle, J28 AVR_SPI_PROG_3X2TESTPOINTS, J3 Qwiic Right Angle, J4 AVR_SPI_PROG_3X2TESTPOINTS, J6 Qwiic Right Angle, J7 Qwiic Right Angle, J8 AVR_SPI_PROG_3X2TESTPOINTS, Q1 600mA/40V, Q2 600mA/40V, Q3 600mA/40V, Q4 600mA/40V, Q5 600mA/40V, Q6 600mA/40V, U1 ATTIN85_SOIC_5.3MM, U10 OPTO_ISOLATOR, U11 ATTIN85_SOIC_5.3MM, U12 OPTO_ISOLATOR, U2 OPTO_ISOLATOR, U3 ATTIN85_SOIC_5.3MM, U4 OPTO_ISOLATOR, U5 ATTIN85_SOIC_5.3MM, U6 OPTO_ISOLATOR, U7 ATTIN85_SOIC_5.3MM, U8 OPTO_ISOLATOR, U9 ATTIN85_SOIC_5.3MM

Commit message: Small changes to silk and version number
Parts:
- added C10, C11, C12, C7, C8, C9: 10uF, SparkFun-Capacitors:0603
- added D19, D22, D25, D28, D31, D34: 1A/23V/620mV, SparkFun-DiscreteSemi:SOD-323
- added D20, D23, D26, D29, D32, D35: BLUE, SparkFun-LED:LED-0603
- added D21, D24, D27, D30, D33, D36: RED, SparkFun-LED:LED-0603
- added J31, J32, J36, J37, J41, J42, J46, J47, J51, J52, J56, J57: Qwiic Right Angle, SparkFun-Connectors:1X04_1MM_RA
- added J33, J38, J43, J48, J53, J58: AVR_SPI_PROG_3X2TESTPOINTS, SparkFun-Connectors:2X3_TEST_POINTS
- added J34, J39, J44, J49, J54, J59: (no value), SparkFun-Connectors:1X04_NO_SILK
- added J35, J40, J45, J50, J55, J60: (no value), SparkFun-Connectors:SCREWTERMINAL-5MM-3
- added JP100, JP110, JP120, JP70, JP80, JP90: JUMPER-SMT_2_NO_NO-SILK, SparkFun-Jumpers:SMT-JUMPER_2_NO_NO-SILK
- added JP101, JP102, JP106, JP107, JP111, JP112, JP116, JP117, JP61, JP62, JP66, JP67, JP71, JP72, JP76, JP77, JP81, JP82, JP86, JP87, JP91, JP92, JP96, JP97: STAND-OFF, SparkFun:STAND-OFF
- added JP103, JP104, JP108, JP109, JP113, JP114, JP118, JP119, JP63, JP64, JP68, JP69, JP73, JP74, JP78, JP79, JP83, JP84, JP88, JP89, JP93, JP94, JP98, JP99: FIDUCIALUFIDUCIAL, SparkFun:MICRO-FIDUCIAL
- added JP105, JP115, JP65, JP75, JP85, JP95: (no value), SparkFun-Jumpers:SMT-JUMPER_3_2-NC_PASTE_SILK
- added K10, K11, K12, K7, K8, K9: (no value), SparkX:RELAY_SPDT_1C
- added LOGO10, LOGO11, LOGO12, LOGO7, LOGO8, LOGO9: OSHW-LOGOMINI, SparkFun-Aesthetics:OSHW-LOGO-MINI
- added Q10, Q11, Q12, Q7, Q8, Q9: 600mA/40V, SparkFun-DiscreteSemi:SOT23-3
- added R49, R57, R65, R73, R81, R89: 10, SparkFun-Resistors:0603
- added R50, R58, R66, R74, R82, R90: 100, SparkFun-Resistors:0603
- added R51, R52, R59, R60, R67, R68, R75, R76, R83, R84, R91, R92: 330, SparkFun-Resistors:0603
- added R53, R54, R61, R62, R69, R70, R77, R78, R85, R86, R93, R94: 2.2K, SparkFun-Resistors:0603
- added R55, R63, R71, R79, R87, R95: 10K, SparkFun-Resistors:0603
- added R56, R64, R72, R80, R88, R96: 1k, SparkFun-Resistors:0603
- added U$103, U$104, U$120, U$121, U$137, U$138, U$154, U$155, U$171, U$172, U$188, U$189: SPARKX-LOGO4, SparkX:SPARKX-MEDIUM
- added U$105, U$122, U$139, U$156, U$173, U$190: (no value), Labels-0_04:(PWR)
- added U$106, U$123, U$140, U$157, U$174, U$191: (no value), Labels-0_04:SCL
- added U$107, U$124, U$141, U$158, U$175, U$192: (no value), Labels-0_04:SDA
- added U$108, U$125, U$142, U$159, U$176, U$193: (no value), Labels-0_04:3.3V
- added U$109, U$126, U$143, U$160, U$177, U$194: (no value), Labels-0_04:GND
- added U$110, U$127, U$144, U$161, U$178, U$195: (no value), buzzard_labels:ACT5
- added U$111, U$112, U$128, U$129, U$145, U$146, U$162, U$163, U$179, U$180, U$196, U$197: (no value), buzzard_labels:QWIIC_RELAY1
- added U$113, U$119, U$130, U$136, U$147, U$153, U$164, U$170, U$181, U$187, U$198, U$204: (no value), buzzard_labels:NC3
- added U$114, U$118, U$131, U$135, U$148, U$152, U$165, U$169, U$182, U$186, U$199, U$203: (no value), buzzard_labels:NO2
- added U$115, U$132, U$149, U$166, U$183, U$200: (no value), buzzard_labels:COM4
- added U$116, U$133, U$150, U$167, U$184, U$201: (no value), Labels-0_04:(ADR)
- added U$117, U$134, U$151, U$168, U$185, U$202: (no value), buzzard_labels (1):COM7
- added U13, U15, U17, U19, U21, U23: ATTIN85_SOIC_5.3MM, attiny85:ATTINY85
- added U14, U16, U18, U20, U22, U24: OPTO_ISOLATOR, SparkX:4PIN_DIP
- moved U$101 100.0 mm to (137.2, -0.38), turned to 90 degrees
- moved U$67 100.0 mm to (85.3, -0.38), turned to 90 degrees
- moved U$84 100.0 mm to (111.3, -0.38), turned to 90 degrees
- moved U$68 99.7 mm to (95.5, -0.13), turned to 90 degrees
- moved U$85 99.7 mm to (121.4, -0.13), turned to 90 degrees
- moved U$102 99.7 mm to (147.3, -0.13), turned to 90 degrees
- moved LOGO4 96.8 mm to (80.1, 11.4), turned to 270 degrees
- moved LOGO5 96.8 mm to (106.0, 11.4), turned to 270 degrees
- moved LOGO6 96.8 mm to (132.0, 11.4), turned to 270 degrees
- moved U$93 96.1 mm to (149.1, 37.3)
- moved U$59 96.1 mm to (97.3, 37.3)
- moved U$76 96.1 mm to (123.2, 37.3)
- moved D11 96.0 mm to (100.6, 41.9)
- moved D14 96.0 mm to (126.5, 41.9)
- moved D16 96.0 mm to (132.1, 38.1)
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Connections:
- new net !RESET10: J53.5, R87.2, U21.1
- new net !RESET11: J58.5, R95.2, U23.1
- new net !RESET6: J33.5, R55.2, U13.1
- new net !RESET7: J38.5, R63.2, U15.1
- new net !RESET8: J43.5, R71.2, U17.1
- new net !RESET9: J48.5, R79.2, U19.1
- new net 3.3V10: C11.1, D32.A, D33.A, J51.2, J52.2, J53.2, J54.3, JP105.2, R81.2, R84.2, R87.1, U21.8
- new net 3.3V11: C12.1, D35.A, D36.A, J56.2, J57.2, J58.2, J59.3, JP115.2, R89.2, R92.2, R95.1, U23.8
- new net 3.3V6: C7.1, D20.A, D21.A, J31.2, J32.2, J33.2, J34.3, JP65.2, R49.2, R52.2, R55.1, U13.8
- new net 3.3V7: C8.1, D23.A, D24.A, J36.2, J37.2, J38.2, J39.3, JP75.2, R57.2, R60.2, R63.1, U15.8
- new net 3.3V8: C9.1, D26.A, D27.A, J41.2, J42.2, J43.2, J44.3, JP85.2, R65.2, R68.2, R71.1, U17.8
- new net 3.3V9: C10.1, D29.A, D30.A, J46.2, J47.2, J48.2, J49.3, JP95.2, R73.2, R76.2, R79.1, U19.8
- new net COM10: J55.2, K11.1
- new net COM11: J60.2, K12.1
- new net COM6: J35.2, K7.1
- new net COM7: J40.2, K8.1
- new net COM8: J45.2, K9.1
- new net COM9: J50.2, K10.1
- new net GND10: C11.2, J51.1, J52.1, J53.6, J54.4, JP110.2, Q11.2, R88.2, U21.4, U22.2
- new net GND11: C12.2, J56.1, J57.1, J58.6, J59.4, JP120.2, Q12.2, R96.2, U23.4, U24.2
- new net GND6: C7.2, J31.1, J32.1, J33.6, J34.4, JP70.2, Q7.2, R56.2, U13.4, U14.2
- new net GND7: C8.2, J36.1, J37.1, J38.6, J39.4, JP80.2, Q8.2, R64.2, U15.4, U16.2
- new net GND8: C9.2, J41.1, J42.1, J43.6, J44.4, JP90.2, Q9.2, R72.2, U17.4, U18.2
- new net GND9: C10.2, J46.1, J47.1, J48.6, J49.4, JP100.2, Q10.2, R80.2, U19.4, U20.2
- new net MISO10: J53.1, U21.6
- new net MISO11: J58.1, U23.6
- new net MISO6: J33.1, U13.6
- new net MISO7: J38.1, U15.6
- new net MISO8: J43.1, U17.6
- new net MISO9: J48.1, U19.6
- new net N$100: JP100.1, U19.2
- new net N$101: D31.A, K11.5, Q11.3, R83.1
- new net N$102: D31.C, K11.2, R81.1
- new net N$103: D32.C, R83.2
- new net N$104: R84.1, U22.4
- new net N$105: JP105.1, R86.2
- new net N$106: JP105.3, R85.2
- new net N$107: D33.C, R88.1
- new net N$108: R82.1, U22.1
- new net N$109: Q11.1, U22.3
- new net N$110: JP110.1, U21.2
- new net N$111: D34.A, K12.5, Q12.3, R91.1
- new net N$112: D34.C, K12.2, R89.1
- new net N$113: D35.C, R91.2
- new net N$114: R92.1, U24.4
- new net N$115: JP115.1, R94.2
- new net N$116: JP115.3, R93.2
- new net N$117: D36.C, R96.1
- new net N$118: R90.1, U24.1
- new net N$119: Q12.1, U24.3
- new net N$120: JP120.1, U23.2
- new net N$61: D19.A, K7.5, Q7.3, R51.1
- new net N$62: D19.C, K7.2, R49.1
- new net N$63: D20.C, R51.2
- new net N$64: R52.1, U14.4
- new net N$65: JP65.1, R54.2
- new net N$66: JP65.3, R53.2
- new net N$67: D21.C, R56.1
- new net N$68: R50.1, U14.1
- new net N$69: Q7.1, U14.3
- new net N$70: JP70.1, U13.2
- new net N$71: D22.A, K8.5, Q8.3, R59.1
- new net N$72: D22.C, K8.2, R57.1
- new net N$73: D23.C, R59.2
- new net N$74: R60.1, U16.4
- new net N$75: JP75.1, R62.2
- new net N$76: JP75.3, R61.2
- new net N$77: D24.C, R64.1
- new net N$78: R58.1, U16.1
- new net N$79: Q8.1, U16.3
- new net N$80: JP80.1, U15.2
- new net N$81: D25.A, K9.5, Q9.3, R67.1
- new net N$82: D25.C, K9.2, R65.1
- new net N$83: D26.C, R67.2
- new net N$84: R68.1, U18.4
- new net N$85: JP85.1, R70.2
- new net N$86: JP85.3, R69.2
- new net N$87: D27.C, R72.1
- new net N$88: R66.1, U18.1
- new net N$89: Q9.1, U18.3
- new net N$90: JP90.1, U17.2
- new net N$91: D28.A, K10.5, Q10.3, R75.1
- new net N$92: D28.C, K10.2, R73.1
- new net N$93: D29.C, R75.2
- new net N$94: R76.1, U20.4
- new net N$95: JP95.1, R78.2
- new net N$96: JP95.3, R77.2
- new net N$97: D30.C, R80.1
- new net N$98: R74.1, U20.1
- new net N$99: Q10.1, U20.3
- new net NC10: J55.1, K11.4
- new net NC11: J60.1, K12.4
- new net NC6: J35.1, K7.4
- new net NC7: J40.1, K8.4
- new net NC8: J45.1, K9.4
- new net NC9: J50.1, K10.4
- new net NO10: J55.3, K11.3
- new net NO11: J60.3, K12.3
- new net NO6: J35.3, K7.3
- new net NO7: J40.3, K8.3
- new net NO8: J45.3, K9.3
- new net NO9: J50.3, K10.3
- new net RELAY_CTR10: R82.2, U21.3
- new net RELAY_CTR11: R90.2, U23.3
- new net RELAY_CTR6: R50.2, U13.3
- new net RELAY_CTR7: R58.2, U15.3
- new net RELAY_CTR8: R66.2, U17.3
- new net RELAY_CTR9: R74.2, U19.3
- new net SCL10: J51.4, J52.4, J53.3, J54.1, R85.1, U21.7
- new net SCL11: J56.4, J57.4, J58.3, J59.1, R93.1, U23.7
- new net SCL6: J31.4, J32.4, J33.3, J34.1, R53.1, U13.7
- new net SCL7: J36.4, J37.4, J38.3, J39.1, R61.1, U15.7
- new net SCL8: J41.4, J42.4, J43.3, J44.1, R69.1, U17.7
- new net SCL9: J46.4, J47.4, J48.3, J49.1, R77.1, U19.7
- new net SDA10: J51.3, J52.3, J53.4, J54.2, R86.1, U21.5
- new net SDA11: J56.3, J57.3, J58.4, J59.2, R94.1, U23.5
- new net SDA6: J31.3, J32.3, J33.4, J34.2, R54.1, U13.5
- new net SDA7: J36.3, J37.3, J38.4, J39.2, R62.1, U15.5
- new net SDA8: J41.3, J42.3, J43.4, J44.2, R70.1, U17.5
- new net SDA9: J46.3, J47.3, J48.4, J49.2, R78.1, U19.5
Routing:
- net 3.3V7: track 0.00 -> 74.1 mm, vias 0 -> 3
- net 3.3V6: track 0.00 -> 74.1 mm, vias 0 -> 3
- net 3.3V9: track 0.00 -> 74.1 mm, vias 0 -> 3
- net 3.3V8: track 0.00 -> 74.1 mm, vias 0 -> 3
- net 3.3V10: track 0.00 -> 74.1 mm, vias 0 -> 3
- net 3.3V11: track 0.00 -> 74.1 mm, vias 0 -> 3
- net COM9: track 0.00 -> 71.3 mm
- net COM8: track 0.00 -> 71.3 mm
- net COM7: track 0.00 -> 71.3 mm
- net COM10: track 0.00 -> 71.3 mm
- net COM6: track 0.00 -> 71.3 mm
- net COM11: track 0.00 -> 71.3 mm
- net SDA10: track 0.00 -> 46.0 mm, vias 0 -> 3
- net SDA6: track 0.00 -> 46.0 mm, vias 0 -> 3
- net SDA7: track 0.00 -> 46.0 mm, vias 0 -> 3
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- added copper zone on layer 1, net GND10
- added copper zone on layer 16, net GND10
- added copper zone on layer 1, net GND11
- added copper zone on layer 16, net GND11
- added copper zone on layer 1, net GND6
- added copper zone on layer 16, net GND6
- added copper zone on layer 1, net GND7
- added copper zone on layer 16, net GND7
- added copper zone on layer 1, net GND8
- added copper zone on layer 16, net GND8
- added copper zone on layer 1, net GND9
- added copper zone on layer 16, net GND9
Other:
- board size 103.1 x 138.2 mm -> 175 x 132.3 mm
- board text added: "route out"
- board text removed: "cutout"

Commit message: Adding Qwiic Logo to bottom silk
Parts:
- added U$205: (no value), Labels-0_04:GND
- added U$206: (no value), buzzard_labels:ACT5
- added U$207, U$208: (no value), buzzard_labels:QWIIC_RELAY1
- added U$209, U$215: (no value), buzzard_labels:NC3
- added U$210, U$214: (no value), buzzard_labels:NO2
- added U$211: (no value), buzzard_labels:COM4
- added U$212: (no value), Labels-0_04:(ADR)
- added U$213: (no value), buzzard_labels (1):COM7
- added U$216: (no value), Labels:QWIIC-LOGO-MEDIUM
- U$1, U$36: value SPARKX-LOGO4 -> (none); device SparkX:SPARKX-MEDIUM -> Labels:QWIIC-LOGO-MEDIUM
- U$100, U$117: device buzzard_labels (1):COM7 -> buzzard_labels:QWIIC_RELAY1
- U$101, U$29: device buzzard_labels:NO2 -> buzzard_labels:NC3
- U$102, U$34: device buzzard_labels:NC3 -> buzzard_labels:NO2
- U$103, U$121: value SPARKX-LOGO4 -> (none); device SparkX:SPARKX-MEDIUM -> buzzard_labels:COM4
- U$104, U$86: value SPARKX-LOGO4 -> (none); device SparkX:SPARKX-MEDIUM -> Labels-0_04:(ADR)
- U$105: device Labels-0_04:(PWR) -> buzzard_labels (1):COM7
- U$106, U$174: device Labels-0_04:SCL -> buzzard_labels:NO2
- U$107: device Labels-0_04:SDA -> buzzard_labels:NC3
- U$108: device Labels-0_04:3.3V -> Labels:QWIIC-LOGO-MEDIUM
- U$109, U$92: value (none) -> SPARKX-LOGO4; device Labels-0_04:GND -> SparkX:SPARKX-MEDIUM
- U$110, U$127: value (none) -> SPARKX-LOGO4; device buzzard_labels:ACT5 -> SparkX:SPARKX-MEDIUM
- U$111, U$129: device buzzard_labels:QWIIC_RELAY1 -> Labels-0_04:(PWR)
- U$112, U$94: device buzzard_labels:QWIIC_RELAY1 -> Labels-0_04:SCL
- U$113: device buzzard_labels:NC3 -> Labels-0_04:SDA
- U$114, U$186: device buzzard_labels:NO2 -> Labels-0_04:3.3V
- U$115: device buzzard_labels:COM4 -> Labels-0_04:GND
- U$116: device Labels-0_04:(ADR) -> buzzard_labels:ACT5
- U$118, U$135, U$46, U$63: device buzzard_labels:NO2 -> buzzard_labels:QWIIC_RELAY1
- U$120, U$138, U$52, U$70: value SPARKX-LOGO4 -> (none); device SparkX:SPARKX-MEDIUM -> buzzard_labels:NO2
- U$122: device Labels-0_04:(PWR) -> Labels-0_04:(ADR)
- U$123: device Labels-0_04:SCL -> buzzard_labels (1):COM7
- U$124, U$192: device Labels-0_04:SDA -> buzzard_labels:NO2
- U$125: device Labels-0_04:3.3V -> buzzard_labels:NC3
- U$126: device Labels-0_04:GND -> Labels:QWIIC-LOGO-MEDIUM
- U$128, U$145, U$146, U$163: value (none) -> SPARKX-LOGO4; device buzzard_labels:QWIIC_RELAY1 -> SparkX:SPARKX-MEDIUM
- U$130: device buzzard_labels:NC3 -> Labels-0_04:SCL
- U$131, U$203: device buzzard_labels:NO2 -> Labels-0_04:SDA
- U$132: device buzzard_labels:COM4 -> Labels-0_04:3.3V
- U$133: device Labels-0_04:(ADR) -> Labels-0_04:GND
- U$134: device buzzard_labels (1):COM7 -> buzzard_labels:ACT5
- U$136, U$153, U$28, U$45: device buzzard_labels:NC3 -> buzzard_labels:QWIIC_RELAY1
- U$137, U$155, U$35, U$53: value SPARKX-LOGO4 -> (none); device SparkX:SPARKX-MEDIUM -> buzzard_labels:NC3
- U$139: device Labels-0_04:(PWR) -> buzzard_labels:COM4
- U$14, U$37: value (none) -> SPARKX-LOGO4; device Labels-0_04:(PWR) -> SparkX:SPARKX-MEDIUM
- U$140: device Labels-0_04:SCL -> Labels-0_04:(ADR)
- U$141: device Labels-0_04:SDA -> buzzard_labels (1):COM7
- U$142: device Labels-0_04:3.3V -> buzzard_labels:NO2
- U$143: device Labels-0_04:GND -> buzzard_labels:NC3
- U$144: device buzzard_labels:ACT5 -> Labels:QWIIC-LOGO-MEDIUM
- U$147: device buzzard_labels:NC3 -> Labels-0_04:(PWR)
- U$148: device buzzard_labels:NO2 -> Labels-0_04:SCL
- U$149: device buzzard_labels:COM4 -> Labels-0_04:SDA
- U$150: device Labels-0_04:(ADR) -> Labels-0_04:3.3V
- U$151: device buzzard_labels (1):COM7 -> Labels-0_04:GND
- U$152, U$80: device buzzard_labels:NO2 -> buzzard_labels:ACT5
- U$154, U$171, U$172, U$189: value SPARKX-LOGO4 -> (none); device SparkX:SPARKX-MEDIUM -> buzzard_labels:QWIIC_RELAY1
- U$156, U$88: device Labels-0_04:(PWR) -> buzzard_labels:NO2
- U$157: device Labels-0_04:SCL -> buzzard_labels:COM4
- U$158: device Labels-0_04:SDA -> Labels-0_04:(ADR)
- U$159: device Labels-0_04:3.3V -> buzzard_labels (1):COM7
- U$160: device Labels-0_04:GND -> buzzard_labels:NO2
- U$161: device buzzard_labels:ACT5 -> buzzard_labels:NC3
- U$162, U$180: device buzzard_labels:QWIIC_RELAY1 -> Labels:QWIIC-LOGO-MEDIUM
- U$164, U$181: value (none) -> SPARKX-LOGO4; device buzzard_labels:NC3 -> SparkX:SPARKX-MEDIUM
- U$165: device buzzard_labels:NO2 -> Labels-0_04:(PWR)
- U$166: device buzzard_labels:COM4 -> Labels-0_04:SCL
- U$167: device Labels-0_04:(ADR) -> Labels-0_04:SDA
- U$168: device buzzard_labels (1):COM7 -> Labels-0_04:3.3V
- U$169, U$97: device buzzard_labels:NO2 -> Labels-0_04:GND
- U$170, U$62: device buzzard_labels:NC3 -> buzzard_labels:ACT5
- U$173, U$71: device Labels-0_04:(PWR) -> buzzard_labels:NC3
- U$175: device Labels-0_04:SDA -> buzzard_labels:COM4
- U$176: device Labels-0_04:3.3V -> Labels-0_04:(ADR)
- U$177: device Labels-0_04:GND -> buzzard_labels (1):COM7
- U$178: device buzzard_labels:ACT5 -> buzzard_labels:NO2
- U$179, U$197: device buzzard_labels:QWIIC_RELAY1 -> buzzard_labels:NC3
- U$182, U$199: value (none) -> SPARKX-LOGO4; device buzzard_labels:NO2 -> SparkX:SPARKX-MEDIUM
- U$183: device buzzard_labels:COM4 -> Labels-0_04:(PWR)
- U$184: device Labels-0_04:(ADR) -> Labels-0_04:SCL
- U$185: device buzzard_labels (1):COM7 -> Labels-0_04:SDA
- U$187, U$79: device buzzard_labels:NC3 -> Labels-0_04:GND
- U$188: value SPARKX-LOGO4 -> (none); device SparkX:SPARKX-MEDIUM -> buzzard_labels:ACT5
- U$190: device Labels-0_04:(PWR) -> buzzard_labels:QWIIC_RELAY1
- U$191, U$89: device Labels-0_04:SCL -> buzzard_labels:NC3
- U$193: device Labels-0_04:3.3V -> buzzard_labels:COM4
- U$194: device Labels-0_04:GND -> Labels-0_04:(ADR)
- U$195: device buzzard_labels:ACT5 -> buzzard_labels (1):COM7
- U$196: device buzzard_labels:QWIIC_RELAY1 -> buzzard_labels:NO2
- U$198: device buzzard_labels:NC3 -> Labels:QWIIC-LOGO-MEDIUM
- U$200: value (none) -> SPARKX-LOGO4; device buzzard_labels:COM4 -> SparkX:SPARKX-MEDIUM
- U$201: device Labels-0_04:(ADR) -> Labels-0_04:(PWR)
- U$202: device buzzard_labels (1):COM7 -> Labels-0_04:SCL
- U$204, U$96: device buzzard_labels:NC3 -> Labels-0_04:3.3V
- U$21: device Labels-0_04:SCL -> Labels-0_04:(PWR)
- U$22: device Labels-0_04:SDA -> Labels-0_04:SCL
- U$23: device Labels-0_04:3.3V -> Labels-0_04:SDA
- U$24: device Labels-0_04:GND -> Labels-0_04:3.3V
- U$25: device buzzard_labels:ACT5 -> Labels-0_04:GND
- U$26, U$44: device buzzard_labels:QWIIC_RELAY1 -> buzzard_labels:ACT5
- U$30: device buzzard_labels:COM4 -> buzzard_labels:NO2
- U$31: device Labels-0_04:(ADR) -> buzzard_labels:COM4
- U$32: device buzzard_labels (1):COM7 -> Labels-0_04:(ADR)
- U$33: device buzzard_labels:NO2 -> buzzard_labels (1):COM7
- U$38, U$55: value (none) -> SPARKX-LOGO4; device Labels-0_04:SCL -> SparkX:SPARKX-MEDIUM
- U$39: device Labels-0_04:SDA -> Labels-0_04:(PWR)
- U$40: device Labels-0_04:3.3V -> Labels-0_04:SCL
- U$41: device Labels-0_04:GND -> Labels-0_04:SDA
- U$42: device buzzard_labels:ACT5 -> Labels-0_04:3.3V
- U$43, U$61: device buzzard_labels:QWIIC_RELAY1 -> Labels-0_04:GND
- U$47: device buzzard_labels:COM4 -> buzzard_labels:NC3
- U$48: device Labels-0_04:(ADR) -> buzzard_labels:NO2
- U$49: device buzzard_labels (1):COM7 -> buzzard_labels:COM4
- U$50: device buzzard_labels:NO2 -> Labels-0_04:(ADR)
- U$51: device buzzard_labels:NC3 -> buzzard_labels (1):COM7
- U$54: device Labels-0_04:(PWR) -> Labels:QWIIC-LOGO-MEDIUM
- U$56, U$73: value (none) -> SPARKX-LOGO4; device Labels-0_04:SDA -> SparkX:SPARKX-MEDIUM
- U$57: device Labels-0_04:3.3V -> Labels-0_04:(PWR)
- U$58: device Labels-0_04:GND -> Labels-0_04:SCL
- U$59: device buzzard_labels:ACT5 -> Labels-0_04:SDA
- U$60, U$78: device buzzard_labels:QWIIC_RELAY1 -> Labels-0_04:3.3V
- U$64, U$81: device buzzard_labels:COM4 -> buzzard_labels:QWIIC_RELAY1
- U$65: device Labels-0_04:(ADR) -> buzzard_labels:NC3
- U$66: device buzzard_labels (1):COM7 -> buzzard_labels:NO2
- U$67: device buzzard_labels:NO2 -> buzzard_labels:COM4
- U$68: device buzzard_labels:NC3 -> Labels-0_04:(ADR)
- U$69, U$87: value SPARKX-LOGO4 -> (none); device SparkX:SPARKX-MEDIUM -> buzzard_labels (1):COM7
- U$72: device Labels-0_04:SCL -> Labels:QWIIC-LOGO-MEDIUM
- U$74, U$91: value (none) -> SPARKX-LOGO4; device Labels-0_04:3.3V -> SparkX:SPARKX-MEDIUM
- U$75: device Labels-0_04:GND -> Labels-0_04:(PWR)
- U$76: device buzzard_labels:ACT5 -> Labels-0_04:SCL
- U$77, U$95: device buzzard_labels:QWIIC_RELAY1 -> Labels-0_04:SDA
- U$82, U$99: device Labels-0_04:(ADR) -> buzzard_labels:QWIIC_RELAY1
- U$83: device buzzard_labels (1):COM7 -> buzzard_labels:NC3
- U$85: device buzzard_labels:NC3 -> buzzard_labels:COM4
- U$90: device Labels-0_04:SDA -> Labels:QWIIC-LOGO-MEDIUM
- U$93: device buzzard_labels:ACT5 -> Labels-0_04:(PWR)
- U$98: device buzzard_labels:COM4 -> buzzard_labels:ACT5
- moved U$107 173.3 mm to (147.3, -0.13), flipped to the top, turned to 90 degrees
- moved U$108 169.1 mm to (151.1, 15.2)
- moved U$105 166.3 mm to (142.2, -0.38)
- moved U$106 163.9 mm to (137.2, -0.38), flipped to the top, turned to 90 degrees
- moved U$103 158.3 mm to (142.4, 8.38), flipped to the bottom, turned to 270 degrees
- moved U$104 155.7 mm to (153.7, 45.8)
- moved U$124 63.3 mm to (7.62, 56.0), flipped to the top, turned to 90 degrees
- moved U$123 62.1 mm to (12.7, 56.0), flipped to the top, turned to 90 degrees
- moved U$142 62.1 mm to (33.5, 56.0), flipped to the top, turned to 90 degrees
- moved U$141 60.9 mm to (38.6, 56.0), flipped to the top, turned to 90 degrees
- moved U$160 60.9 mm to (59.4, 56.0), flipped to the top, turned to 90 degrees
- moved U$159 59.8 mm to (64.5, 56.0), flipped to the top, turned to 90 degrees
- moved U$89 59.6 mm to (121.4, -0.13), flipped to the top, turned to 90 degrees
- moved U$177 58.8 mm to (90.4, 56.0), flipped to the top, turned to 90 degrees
- moved U$125 57.6 mm to (17.8, 56.3), flipped to the top, turned to 90 degrees
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